Commit message: Adjust the controller nlaunnch file

File: src/robokrub_description/urdf/robokrub.xacro (robot description, xacro)
@@ -1,4 +1,4 @@
 <?xml version="1.0" ?>
-<robot name="robokrub" xmlns:xacro="http://www.ros.org/wiki/xacro">
+<robot name="walkie" xmlns:xacro="http://www.ros.org/wiki/xacro">
 <xacro:include filename="$(find robokrub_description)/urdf/materials.xacro" />
 <xacro:include filename="$(find robokrub_description)/urdf/robokrub.trans" />
@@ -176,4 +176,5 @@
   <child link="realsense_base_1"/>
   <axis xyz="-0.000175 0.002437 -0.999997"/>
+  <dynamics damping="0.0"/>
 </joint>
 <joint name="realsense_roll_joint" type="continuous">
@@ -182,4 +183,5 @@
   <child link="realsense_mount_1"/>
   <axis xyz="-0.004129 0.999989 0.002438"/>
+  <dynamics damping="0.0"/>
 </joint>
 <joint name="left_back_wheel_joint" type="continuous">

Commit message: Add controllers and realsense to original URDF

File: src/robokrub_description/urdf/robokrub.xacro (robot description, xacro)
@@ -171,5 +171,5 @@
   </collision>
 </link>
-<joint name="realsense_pitch_joint" type="continuous">
+<joint name="realsense_yaw_joint" type="continuous">
   <origin rpy="0 0 0" xyz="-0.043071 -0.002012 1.303319"/>
   <parent link="base_link"/>
@@ -178,5 +178,5 @@
   <dynamics damping="0.0"/>
 </joint>
-<joint name="realsense_roll_joint" type="continuous">
+<joint name="realsense_pitch_joint" type="continuous">
   <origin rpy="0 0 0" xyz="0.01485 0.061768 0.028648"/>
   <parent link="realsense_base_1"/>
@@ -212,3 +212,8 @@
   <child link="Hokuyo_UST-10LX__2__v1_1"/>
 </joint>
+<xacro:include filename="$(find simplify_description)/urdf/_d435.urdf.xacro" />
+<xacro:sensor_d435 name="sensor_d435" parent="realsense_mount_1">
+    <origin xyz="0.01 -0.06 -0.01" rpy="0 0 0"/>
+    <!-- <origin xyz="0 0 0" rpy="${-90.0 * deg_to_rad} 0 ${-90.0 * deg_to_rad}"/> -->
+</xacro:sensor_d435>
 </robot>

File: src/walkie_simplify_v3/urdf/_d435.urdf.xacro (robot description, xacro)
@@ -9,5 +9,5 @@
   <!--File includes-->
   <xacro:include filename="$(find simplify_description)/urdf/_d435.gazebo.xacro"/>
-  <xacro:macro name="sensor_d435" params="name:=camera topics_ns:=camera parent *origin">
+  <xacro:macro name="sensor_d435" params="name:=camera topics_ns:=walkie/camera parent *origin">
     <xacro:property name="M_PI" value="3.1415926535897931" />
     <!-- The following values are approximate, and the camera node

Commit message: Add planar move and fake human object + new map

File: src/robokrub_description/urdf/robokrub.xacro (robot description, xacro)
@@ -212,8 +212,7 @@
   <child link="Hokuyo_UST-10LX__2__v1_1"/>
 </joint>
-<xacro:include filename="$(find simplify_description)/urdf/_d435.urdf.xacro" />
+<!-- <xacro:include filename="$(find simplify_description)/urdf/_d435.urdf.xacro" />
 <xacro:sensor_d435 name="sensor_d435" parent="realsense_mount_1">
     <origin xyz="0.01 -0.06 -0.01" rpy="0 0 0"/>
-    <!-- <origin xyz="0 0 0" rpy="${-90.0 * deg_to_rad} 0 ${-90.0 * deg_to_rad}"/> -->
-</xacro:sensor_d435>
+</xacro:sensor_d435> -->
 </robot>

Commit message: arch update

File: src/robokrub_description/urdf/robokrub.xacro (robot description, xacro)
@@ -212,4 +212,10 @@
   <child link="Hokuyo_UST-10LX__2__v1_1"/>
 </joint>
+<joint name="imu_joint" type="fixed">
+    <parent link="base_link"/>
+    <child link="imu_link"/>
+    <origin xyz="0 0 0" rpy="0 0 0"/>
+  </joint>
+  <link name="imu_link"/>
 <!-- <xacro:include filename="$(find simplify_description)/urdf/_d435.urdf.xacro" />
 <xacro:sensor_d435 name="sensor_d435" parent="realsense_mount_1">
